Commit message: kure avare

File: myrobot_description/urdf/caster_wheel.urdf.xacro (robot description, xacro)
@@ -4,65 +4,24 @@
  <xacro:property name="caster_wheel_length" value="0.04"/>
 <xacro:macro name="caster_wheel">
-        <link name="caster_wheel">
-         <xacro:cylinder_inertia m="1" r="${caster_wheel_radius}" h="${caster_wheel_length}"/>
-            <visual>
-                <origin xyz="0 0 0" rpy="1.57 0 0"/>
-                <geometry>
-                    <cylinder radius="${caster_wheel_radius}" length="${caster_wheel_length}"/>
-                </geometry>
-                </visual>
-            <collision>
-                <origin xyz="0 0 0" rpy="1.57 0 0"/>
-                <geometry>
-                    <cylinder radius="${caster_wheel_radius}" length="${caster_wheel_length}"/>
-                </geometry>
-            </collision>
-        </link>
-        <link name="caster_fixed">
-        <xacro:box_inertia m="0.1" w="0.1" h="0.1" d="0.1"/>
-            <visual>
-                <origin xyz="0 0 0" rpy="0 0 0"/>
-                <geometry>
-                    <box size="0.01 0.01 0.01"/>
-                </geometry>
-                </visual>
-            <collision>
-                <origin xyz="0 0 0" rpy= "0 0 0"/>
-                <geometry>
-                    <box size="0.01 0.01 0.01"/>
-                </geometry>
-            </collision>
-        </link>
-        <link name="caster_top">
-        <xacro:box_inertia m="0.1" w="0.1" h="0.1" d="0.1"/>
-            <visual>
-                <origin xyz="0 0 0" rpy="0 0 0"/>
-                <geometry>
-                    <box size="0.01 0.01 0.01"/>
-                </geometry>
-                </visual>
-            <collision>
-                <origin xyz="0 0 0" rpy= "0 0 0"/>
-                <geometry>
-                    <box size="0.01 0.01 0.01"/>
-                </geometry>
-            </collision>
-        </link>
-    <joint name="caster_wheel_joint" type="continuous">
-        <axis xyz="0 1 0" rpy="0 0 0"/>
-        <parent link="caster_fixed"/>
+    <link name="caster_wheel">
+        <xacro:box_inertia m="1" w="0.1" h="0.1" d="0.1"/>
+        <visual>
+            <geometry>
+                <sphere radius="0.1"/>
+            </geometry>
+            <material name="orange"/>
+        </visual>
+        <collision>
+            <geometry>
+                <sphere radius="0.1"/>
+            </geometry>
+        </collision>
+    </link>
+    <joint name="caster_joint" type="fixed">
+        <origin xyz="-0.3 0 ${-(base_height/2)}" rpy="0 0 0"/>
+        <parent link="base_link"/>
         <child link="caster_wheel"/>
-        <origin xyz="0 0 ${-caster_wheel_radius}" rpy="0 0 0"/>
-    </joint>
-    <joint name="caster_fixed_joint" type="fixed">
-        <parent link="caster_top"/>
-        <child link="caster_fixed"/>
-        <origin xyz="0 0 -0.005" rpy="0 0 0"/>
-    </joint>
-    <joint name="caster_top_joint" type="continuous">
-        <axis xyz="0 0 1" rpy="0 0 0"/>
-        <parent link="base_link"/>
-        <child link="caster_top"/>
-        <origin xyz="-0.3 0 ${-(base_height/2) - 0.005}" rpy="0 0 0"/>
+        <calibration rising="0.0"/>
+        <dynamics damping="0.0" friction="0.0"/>
     </joint>
     </xacro:macro>

File: myrobot_description/urdf/caster_wheel/caster_wheel.urdf.xacro (robot description, xacro)
@@ -1,66 +1,69 @@
 <?xml version="1.0"?>
 <robot xmlns:xacro="http://www.ros.org/wiki/xacro" name="wheel">
-<xacro:property name="caster_wheel_radius" value="0.01"/>
-<xacro:property name="caster_wheel_length" value="0.04"/>
+ <xacro:property name="caster_wheel_radius" value="0.01"/>
+ <xacro:property name="caster_wheel_length" value="0.04"/>
 <xacro:macro name="caster_wheel">
-    <link name="caster_wheel">
-        <visual>
-            <origin xyz="0 0 0" rpy="1.57 0 0"/>
-            <geometry>
-                <cylinder radius="${caster_wheel_radius}" length="${caster_wheel_length}"/>
-            </geometry>
-            </visual>
-        <collision>
-            <origin xyz="0 0 0" rpy="1.57 0 0"/>
-            <geometry>
-                <cylinder radius="${caster_wheel_radius}" length="${caster_wheel_length}"/>
-            </geometry>
-        </collision>
-    </link>
-    <link name="caster_fixed">
-        <visual>
-            <origin xyz="0 0 0" rpy="0 0 0"/>
-            <geometry>
-                <box size="0.01 0.01 0.01"/>
-            </geometry>
-            </visual>
-        <collision>
-            <origin xyz="0 0 0" rpy= "0 0 0"/>
-            <geometry>
-                <box size="0.01 0.01 0.01"/>
-            </geometry>
-        </collision>
-    </link>
-    <link name="caster_top">
-        <visual>
-            <origin xyz="0 0 0" rpy="0 0 0"/>
-            <geometry>
-                <box size="0.01 0.01 0.01"/>
-            </geometry>
-            </visual>
-        <collision>
-            <origin xyz="0 0 0" rpy= "0 0 0"/>
-            <geometry>
-                <box size="0.01 0.01 0.01"/>
-            </geometry>
-        </collision>
-    </link>
-<joint name="caster_wheel_joint" type="continuous">
-    <axis xyz="0 1 0" rpy="0 0 0"/>
-    <parent link="caster_fixed"/>
-    <child link="caster_wheel"/>
-    <origin xyz="0 0 0" rpy="0 0 0"/>
-</joint>
-<joint name="caster_fixed_joint" type="fixed">
-    <parent link="caster_top"/>
-    <child link="caster_fixed"/>
-    <origin xyz="0 0 0" rpy="0 0 0"/>
-</joint>
-<joint name="caster_top_joint" type="continuous">
-    <axis xyz="0 0 1" rpy="0 0 0"/>
-    <parent link="base_link"/>
-    <child link="caster_top"/>
-    <origin xyz="0 0 ${(base_height/2) - base_distance_from_ground}" rpy="0 0 0"/>
-</joint>
-</xacro:macro>
+        <link name="caster_wheel">
+         <xacro:cylinder_inertia m="1" r="${caster_wheel_radius}" h="${caster_wheel_length}"/>
+            <visual>
+                <origin xyz="0 0 0" rpy="1.57 0 0"/>
+                <geometry>
+                    <cylinder radius="${caster_wheel_radius}" length="${caster_wheel_length}"/>
+                </geometry>
+                </visual>
+            <collision>
+                <origin xyz="0 0 0" rpy="1.57 0 0"/>
+                <geometry>
+                    <cylinder radius="${caster_wheel_radius}" length="${caster_wheel_length}"/>
+                </geometry>
+            </collision>
+        </link>
+        <link name="caster_fixed">
+        <xacro:box_inertia m="0.1" w="0.1" h="0.1" d="0.1"/>
+            <visual>
+                <origin xyz="0 0 0" rpy="0 0 0"/>
+                <geometry>
+                    <box size="0.01 0.01 0.01"/>
+                </geometry>
+                </visual>
+            <collision>
+                <origin xyz="0 0 0" rpy= "0 0 0"/>
+                <geometry>
+                    <box size="0.01 0.01 0.01"/>
+                </geometry>
+            </collision>
+        </link>
+        <link name="caster_top">
+        <xacro:box_inertia m="0.1" w="0.1" h="0.1" d="0.1"/>
+            <visual>
+                <origin xyz="0 0 0" rpy="0 0 0"/>
+                <geometry>
+                    <box size="0.01 0.01 0.01"/>
+                </geometry>
+                </visual>
+            <collision>
+                <origin xyz="0 0 0" rpy= "0 0 0"/>
+                <geometry>
+                    <box size="0.01 0.01 0.01"/>
+                </geometry>
+            </collision>
+        </link>
+    <joint name="caster_wheel_joint" type="continuous">
+        <axis xyz="0 1 0" rpy="0 0 0"/>
+        <parent link="caster_fixed"/>
+        <child link="caster_wheel"/>
+        <origin xyz="0 0 ${-caster_wheel_radius}" rpy="0 0 0"/>
+    </joint>
+    <joint name="caster_fixed_joint" type="fixed">
+        <parent link="caster_top"/>
+        <child link="caster_fixed"/>
+        <origin xyz="0 0 -0.005" rpy="0 0 0"/>
+    </joint>
+    <joint name="caster_top_joint" type="continuous">
+        <axis xyz="0 0 1" rpy="0 0 0"/>
+        <parent link="base_link"/>
+        <child link="caster_top"/>
+        <origin xyz="-0.3 0 ${-(base_height/2) - 0.005}" rpy="0 0 0"/>
+    </joint>
+    </xacro:macro>
 </robot>

File: myrobot_description/urdf/myrobot.urdf.xacro (robot description, xacro)
@@ -1,61 +1,62 @@
 <?xml version="1.0"?>
 <robot xmlns:xacro="http://www.ros.org/wiki/xacro" name="myrobot">
-<xacro:property name="base_width" value="1"/>
-<xacro:property name="base_len" value="1"/>
-<xacro:property name="base_height" value="0.5"/>
-<xacro:property name="base_distance_from_ground" value="0.03"/>
-<xacro:include filename="$(find myrobot_description)/urdf/robot.gazebo"/>
-<!--Color Properties-->
-  <material name="blue">
-    <color rgba="0 0 0.8 1"/>
-  </material>
-  <material name="black">
-    <color rgba="0 0 0 1"/>
-  </material>
-  <material name="white">
-    <color rgba="1 1 1 1"/>
-  </material>
-  <material name="orange">
-    <color rgba="0.5 0.2 0.2 1"/>
-  </material>
-  <!--Interial macros-->
-  <xacro:macro name="cylinder_inertia" params="m r h">
-    <inertial>
-      <mass value="${m}"/>
-      <inertia ixx="${m*(3*r*r+h*h)/12}" ixy = "0" ixz = "0" iyy="${m*(3*r*r+h*h)/12}" iyz = "0" izz="${m*r*r/2}"/>
-    </inertial>
-  </xacro:macro>
-  <xacro:macro name="box_inertia" params="m w h d">
-    <inertial>
-      <mass value="${m}"/>
-      <inertia ixx="${m / 12.0 * (d*d + h*h)}" ixy="0.0" ixz="0.0" iyy="${m / 12.0 * (w*w + h*h)}" iyz="0.0" izz="${m / 12.0 * (w*w + d*d)}"/>
-    </inertial>
-  </xacro:macro>
-<link name="base_link">
-    <xacro:box_inertia m="1" w="${base_len}" h="${base_width}" d="${base_height}"/>
-    <visual>
-        <geometry>
-            <box size="${base_width} ${base_len} ${base_height}"/>
-        </geometry>
-        <material name="blue"/>
-    </visual>
-    <collision>
-        <geometry>
-            <box size="${base_width} ${base_len} ${base_height}"/>
-        </geometry>
-    </collision>
-</link>
-<link name="base_footprint"/>
-  <joint name="base_footprint_joint" type="fixed">
-    <origin xyz="0 0 ${0 - base_distance_from_ground - base_height/2}" rpy="0 0 0" />
-    <parent link="base_link"/>
-    <child link="base_footprint"/>
-  </joint>
-<xacro:include filename="$(find myrobot_description)/urdf/wheel.urdf.xacro"/>
-<xacro:wheel prefix="right" reflect="-1"/>
-<xacro:wheel prefix="left" reflect="1"/>
-<xacro:include filename="$(find myrobot_description)/urdf/caster_wheel.urdf.xacro"/>
-<xacro:caster_wheel/>
-<xacro:include filename="$(find myrobot_description)/urdf/laser_scanner.urdf.xacro"/>
-<xacro:laser_scanner/>
+    <xacro:property name="base_width" value="1"/>
+    <xacro:property name="base_len" value="1"/>
+    <xacro:property name="base_height" value="0.5"/>
+    <xacro:property name="base_distance_from_ground" value="0.1"/>
+    <xacro:include filename="$(find myrobot_description)/urdf/robot.gazebo"/>
+    <!--Color Properties-->
+    <material name="blue">
+        <color rgba="0 0 0.8 1"/>
+    </material>
+    <material name="black">
+        <color rgba="0 0 0 1"/>
+    </material>
+    <material name="white">
+        <color rgba="1 1 1 1"/>
+    </material>
+    <material name="orange">
+        <color rgba="0.5 0.2 0.2 1"/>
+    </material>
+    <!--Interial macros-->
+    <xacro:macro name="cylinder_inertia" params="m r h">
+        <inertial>
+            <mass value="${m}"/>
+            <inertia ixx="${m*(3*r*r+h*h)/12}" ixy="0" ixz="0" iyy="${m*(3*r*r+h*h)/12}" iyz="0" izz="${m*r*r/2}"/>
+        </inertial>
+    </xacro:macro>
+    <xacro:macro name="box_inertia" params="m w h d">
+        <inertial>
+            <mass value="${m}"/>
+            <inertia ixx="${m / 12.0 * (d*d + h*h)}" ixy="0.0" ixz="0.0" iyy="${m / 12.0 * (w*w + h*h)}" iyz="0.0"
+                     izz="${m / 12.0 * (w*w + d*d)}"/>
+        </inertial>
+    </xacro:macro>
+    <link name="base_link">
+        <xacro:box_inertia m="1" w="${base_len}" h="${base_width}" d="${base_height}"/>
+        <visual>
+            <geometry>
+                <box size="${base_width} ${base_len} ${base_height}"/>
+            </geometry>
+            <material name="blue"/>
+        </visual>
+        <collision>
+            <geometry>
+                <box size="${base_width} ${base_len} ${base_height}"/>
+            </geometry>
+        </collision>
+    </link>
+    <link name="base_footprint"/>
+    <joint name="base_footprint_joint" type="fixed">
+        <origin xyz="0 0 ${0 - base_distance_from_ground - base_height/2}" rpy="0 0 0"/>
+        <parent link="base_link"/>
+        <child link="base_footprint"/>
+    </joint>
+    <xacro:include filename="$(find myrobot_description)/urdf/wheel.urdf.xacro"/>
+    <xacro:wheel prefix="right" reflect="-1"/>
+    <xacro:wheel prefix="left" reflect="1"/>
+    <xacro:include filename="$(find myrobot_description)/urdf/caster_wheel.urdf.xacro"/>
+    <xacro:caster_wheel/>
+    <xacro:include filename="$(find myrobot_description)/urdf/laser_scanner.urdf.xacro"/>
+    <xacro:laser_scanner/>
 </robot>
