Commit message: msgs

File: myrobot_description/urdf/myrobot.urdf.xacro (robot description, xacro)
@@ -2,5 +2,5 @@
 <robot xmlns:xacro="http://www.ros.org/wiki/xacro" name="myrobot">
     <xacro:property name="base_width" value="1"/>
-    <xacro:property name="base_len" value="1"/>
+    <xacro:property name="base_len" value="0.6"/>
     <xacro:property name="base_height" value="0.2"/>
     <xacro:property name="base_distance_from_ground" value="0.05"/>

File: myrobot_description/urdf/wheel.urdf.xacro (robot description, xacro)
@@ -23,5 +23,5 @@
             <parent link="base_link"/>
             <child link="${prefix}_wheel"/>
-            <origin xyz="${0.3 * reflect_x} ${(base_width/2 + wheel_length/2) * reflect_y} ${wheel_radius - base_distance_from_ground - (base_height/2)}"
+            <origin xyz="${0.3 * reflect_x} ${(base_len/2 + wheel_length/2) * reflect_y} ${wheel_radius - base_distance_from_ground - (base_height/2)}"
                     rpy="0 0 0"/>
         </joint>

Commit message: lifting eklenmesi

File: myrobot_description/urdf/myrobot.urdf.xacro (robot description, xacro)
@@ -62,3 +62,44 @@
     <xacro:include filename="$(find myrobot_description)/urdf/camera.urdf.xacro"/>
     <xacro:camera_link/>
+    <link name="elevator">
+    <inertial>
+        <origin rpy="0 0 0" xyz="-2.7755575615628914e-15 -0.0022800822836666623 0.09050102854580892"/>
+        <mass value="8.994467062407036"/>
+        <inertia ixx="0.120393" ixy="-0.0" ixz="-0.0" iyy="0.325419" iyz="0.000697" izz="0.415842"/>
+    </inertial>
+    <visual>
+        <origin rpy="0 0 0" xyz="-0.5 -0.305 -0.075"/>
+        <geometry>
+        <mesh filename="package://myrobot_description/meshes/elevator_1.stl" scale="0.001 0.001 0.001"/>
+        </geometry>
+        <material name="red"/>
+    </visual>
+    <collision>
+        <origin rpy="0 0 0" xyz="-0.5 -0.305 -0.075"/>
+        <geometry>
+        <mesh filename="package://myrobot_description/meshes/elevator_1.stl" scale="0.001 0.001 0.001"/>
+        </geometry>
+    </collision>
+    </link>
+    <joint name="slider" type="prismatic">
+    <origin rpy="0 0 0" xyz="0.0 0.0 -0.025"/>
+    <parent link="base_link"/>
+    <child link="elevator"/>
+    <axis xyz="0.0 0.0 1.0"/>
+    <limit effort="100" lower="0.0" upper="0.1" velocity="100"/>
+    </joint>
+	<!-- Transmission is important to link the joints and the controller (see rb1_control/config/rb1_control.yaml)-->
+		<transmission name="elevator_platform_trans">
+			<type>transmission_interface/SimpleTransmission</type>
+			<joint name="slider">
+				<!-- for the gazebo plugin -->
+				<!--hardwareInterface>EffortJointInterface</hardwareInterface-->
+				<!-- for ros control controller -->
+				<hardwareInterface>hardware_interface/EffortJointInterface</hardwareInterface>
+			</joint>
+			<actuator name="elevator_platform_joint_motor">
+				<hardwareInterface>EffortJointInterface</hardwareInterface>
+				<mechanicalReduction>1</mechanicalReduction>
+			</actuator>
+		</transmission>
 </robot>

Commit message: elevator eklendi

File: myrobot_description/urdf/myrobot.urdf.xacro (robot description, xacro)
@@ -82,22 +82,22 @@
     </collision>
     </link>
-    <joint name="slider" type="prismatic">
+    <joint name="elevator_joint" type="prismatic">
     <origin rpy="0 0 0" xyz="0.0 0.0 -0.025"/>
     <parent link="base_link"/>
     <child link="elevator"/>
     <axis xyz="0.0 0.0 1.0"/>
-    <limit effort="100" lower="0.0" upper="0.1" velocity="100"/>
+    <limit effort="100" lower="0.0" upper="0.1" velocity="0.5"/>
     </joint>
 	<!-- Transmission is important to link the joints and the controller (see rb1_control/config/rb1_control.yaml)-->
 		<transmission name="elevator_platform_trans">
 			<type>transmission_interface/SimpleTransmission</type>
-			<joint name="slider">
+			<joint name="elevator_joint">
 				<!-- for the gazebo plugin -->
 				<!--hardwareInterface>EffortJointInterface</hardwareInterface-->
 				<!-- for ros control controller -->
-				<hardwareInterface>hardware_interface/EffortJointInterface</hardwareInterface>
+				<hardwareInterface>hardware_interface/VelocityJointInterface</hardwareInterface>
 			</joint>
 			<actuator name="elevator_platform_joint_motor">
-				<hardwareInterface>EffortJointInterface</hardwareInterface>
+				<hardwareInterface>hardware_interface/VelocityJointInterface</hardwareInterface>
 				<mechanicalReduction>1</mechanicalReduction>
 			</actuator>
